File: Hardware/Iguana_V1/Iguana_V1.kicad_pcb (KiCad board)
At the start: 2 copper layers, 80 x 50 mm, 112 parts, among them J1 BAT, J10 OLED, J11 rgb led, J12 USB_B_Micro, J13 HDR-2x1, J14 Conn_01x02, J17 Conn_Coaxial, J18 IN, J19 IN, J2 HDR-2x1, J3 IN, J4 Cap. Moisture Sensor, J5 ds18b20, J6 SHT31, J7 NPK/H Sensor, J8 ON OFF, J9 HDR-3x1, Q1 Q_PMOS_GSD, Q2 Q_PMOS_GSD, Q3 Q_Dual_NPN_NPN_BRT_E1B1C2E2B2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, Q4 BSS138, SW1 SW_DIP_x02, SW2 SW_DIP_x02, SW3 SW_DIP_x02, U1 DW01, U10 ESP32-WROOM-32D, U11 RV-8803, U12 RFM95W-915S2, U2 TP4056, U3 MT3608, U4 FS8205A, U5 AP2112K-3.3, U6 AP2112K-3.3, U7 MAX3485, U8 AP2112K-3.3, U9 CH340C

Commit message: pcb finished
Parts:
- added G***: LOGO, IoWLabsLogos:iguana_20mm, F.Cu at (126.0, 47.7)
- added G***: LOGO, IoWLabsLogos:iguana_logo, F.Cu at (113.7, 47.5)
- added G***: LOGO, IoWLabsLogos:IoWLabs_logo_13mm, F.Cu at (104.6, 66.9)
- added G***: LOGO, IoWLabsLogos:iguana_logo, B.Cu at (96.4, 39.3)
- added G***: LOGO, IoWLabsLogos:IoWLabs_logo_13mm, B.Cu at (95.8, 46.9)
- added G***: LOGO, IoWLabsLogos:iguana_15mm, B.Cu at (151.7, 57.6)
- added REF**: OSHW-Logo2_9.8x8mm_SilkScreen, Symbol:OSHW-Logo2_9.8x8mm_SilkScreen, F.Cu at (124.2, 58.5)
- added REF**: OSHW-Logo2_9.8x8mm_SilkScreen, Symbol:OSHW-Logo2_9.8x8mm_SilkScreen, B.Cu at (89.5, 53.8)
- moved R15 1.81 mm to (89.1, 42.0)
- moved R8 0.05 mm to (116.2, 56.8)
Connections:
- U10 pad 13: /RBG -> /RGB
Routing:
- net /BAT_LVL: track 1.60 -> 67.7 mm, vias 0 -> 1
- net /RGB: track 19.5 -> 66.4 mm, vias 0 -> 1
- net /VS_3V3: track 112.3 -> 152.5 mm, vias 2 -> 3
- net +5V: track 116.9 -> 150.5 mm, vias 3 -> 4
- net /SPI1_MOSI: track 41.5 -> 67.6 mm, vias 1 -> 2
- net /LORA_CS: track 25.4 -> 45.4 mm, vias 0 -> 1
- net /SPI1_MISO: track 36.1 -> 54.4 mm
- net /SPI1_CLK: track 36.8 -> 54.8 mm
- net /RBG: track 14.9 -> 0.00 mm
- net GND: track 15.8 -> 26.7 mm, vias 27 -> 157
- net /IO2: track 0.11 -> 3.36 mm
- net /LORA_RST: track 38.9 -> 41.8 mm
- net /RS485_RX: track 53.0 -> 55.5 mm
- net +3V3: track 173.9 -> 176.2 mm
- net /IO0: track 29.7 -> 27.7 mm
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Other:
- board text added: "3.3v"
- board text added: "5v"
- board text added: "Iguana board v1.0.0 10/23"
- board text added: "Moisture"
- board text added: "OLED"
- board text added: "ON/OFF"
- board text added: "RGB"
- board text added: "SHT3x"
- board text added: "Temperature"
- board text added: "boot"
- board text added: "rst"
