File: hardware/PCB/Iguana_V1.kicad_sch (KiCad schematic)
At the start: 112 parts, among them J1 BAT, J10 OLED, J11 rgb led, J12 USB_B_Micro, J13 HDR-2x1, J14 Conn_01x02, J17 Conn_Coaxial, J18 IN, J19 IN, J2 HDR-2x1, J3 IN, J4 Cap. Moisture Sensor, J5 ds18b20, J6 SHT31, J7 NPK/H Sensor, J8 ON OFF, J9 HDR-3x1, Q1 Q_PMOS_GSD, Q2 Q_PMOS_GSD, Q3 Q_Dual_NPN_NPN_BRT_E1B1C2E2B2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, Q4 BSS138, SW1 SW_DIP_x02, SW2 SW_DIP_x02, SW3 SW_DIP_x02, U1 DW01, U10 ESP32-WROOM-32D, U11 RV-8803, U12 RFM95W-915S2, U2 TP4056, U3 MT3608, U4 FS8205A, U5 AP2112K-3.3, U6 AP2112K-3.3, U7 MAX3485, U8 AP2112K-3.3, U9 CH340C

Commit message: organizing the schematic. firmware lib v1 working.
Other:
- note added: "Connectors"
- note added: "MODBUS SENSOR"
- note added: "OLED DISPLAY"
- note added: "PUMP"
- note added: "Pump driver"
- note added: "RGB LED"
- note added: "RS485 converter"
- note added: "Tabla de pines ---------------- SPI1_MOSI - GPIO23 SPI1_MISO - GPIO19 SPI1_SCK - GPIO18 CS_SD - GPIO5 RGB - GPIO14 PUMP - GPIO13 LORA_CS - GPIO15 LORA_RST - GPIO25 LORA_D0 - GPIO26 LORA_D1 - GPIO27 I2C_SDA - GPIO21 I2C_SCL - GPIO22 RS485_TX - GPIO16 RS485_Rx - GPIO17 RS485_EN - GPIO4 SENS_M - GPIO34 SENS_TEMP - GPIO32 EN_V - GPIO33 BAT_LVL - GPIO35"
- note removed: "Tabla de pines ---------------- SPI1_MOSI - GPIO23 SPI1_MISO - GPIO19 SPI1_SCK - GPIO18 CS_SD - GPIO5 RGB - GPIO13 - GPIO12 PUMP - GPIO14 LORA_CS - GPIO15 LORA_RST - GPIO25 LORA_D0 - GPIO26 LORA_D1 - GPIO27 I2C_SDA - GPIO21 I2C_SCL - GPIO22 RS485_TX - GPIO16 RS485_Rx - GPIO17 RS485_EN - GPIO4 SENS_M - GPIO34 SENS_TEMP - GPIO32 EN_VDL - GPIO33 EN_VS - GPIO33"
- moved on the sheet: BT1, C1, C10, C11, C12, C13, C14, C15, C16, C17, C18, C19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
